File: KICAD-Boat-Diagnostics/KICAD-Boat-Diagnostics.kicad_pcb (KiCad board)
At the start: 2 copper layers, 1 part, among them U1 ESP32-WROOM-32E_(16MB)

Commit message: Added Power ports
Connections:
- net Net-(U1-Pad1) renamed GND
- net Net-(U1-Pad2) renamed +3V3
